File: TTL/schematic/ALUREGS/ALUREGS.sch (KiCad schematic (older format))
At the start: 7 parts

Commit message: Added docu, work in progress schematics and vhdl
Parts:
- removed U? (x7): 74LS189, symbol TTL:74LS189
- added U? (x2): 74LS175, symbol 74xx:74LS175
- added U? (x2): 74LS283, symbol 74xx:74LS283
- added U? (x2): 74LS153, symbol 74xx:74LS153
- added U? (x3): 74LS157, symbol 74xx:74LS157
- added U?: 74LS74, symbol 74xx:74LS74
- added U? (x2): 74LS08, symbol 74xx:74LS08
- added U? (x2): 74LS32, symbol 74xx:74LS32
- added U?: 8k x 8 SRAM, Package_DIP:DIP-28_W15.24mm, symbol Memory_NVRAM:FM16W08-SG
- added U? (x2): 74LS11, symbol 74xx:74LS11
- added U?: 74LS191, symbol 74xx:74LS191
- added U?: 74LS393, symbol 74xx:74LS393
- added U?: 74LS138, symbol 74xx:74LS138
- added U? (x2): 74LS574, symbol 74xx:74LS574
Connections:
- net labels added: alu_left[0], alu_left[1], alu_left[2], alu_left[3], alu_left_pre[0], alu_left_pre[1], alu_left_pre[2], alu_left_pre[3], alu_left_pre_n[0], alu_left_pre_n[1], alu_left_pre_n[2], alu_left_pre_n[3], alu_right[0], alu_right[1], alu_right[2], alu_right[3], alu_right_pre[0], alu_right_pre[1], alu_right_pre[2], alu_right_pre[3], alu_right_pre_n[0], alu_right_pre_n[1], alu_right_pre_n[2], alu_right_pre_n[3], binadd_q[0], binadd_q[1], binadd_q[2], binadd_q[3], decimal_adjust, dst_r[0], dst_r[1], dst_r[2], dst_r[3], imux_q[0], imux_q[1], imux_q[2], imux_q[3], op1_r[0], op1_r[1], op1_r[2], op1_r[3], regs_a[4], regs_a[5], regs_a[6], regs_a[7]
- net labels removed: regs_a[0], regs_imux[0], regs_imux[1], regs_imux[2], regs_imux[3], regs_q[0], regs_q[1], regs_q[2], regs_q[3], ~reg_a_cs, ~reg_a_we
- wire segments 98 -> 201
Other:
- note added: "OP1 / Destination register/mux"
- note added: "Sequencer"
- note removed: "REG A"
- note removed: "REG B"
- note removed: "REG C"
- note removed: "REG T"
- note removed: "REG Y"
- note removed: "REG Z"
